File: No MCU Sequencer/ELEC 240 Project.kicad_sch (KiCad schematic)
At the start: 34 parts, among them Q4 NMOS, Q5 NMOS, Q6 NMOS, SW2 MODE, SW3 RECORD, SW7 Note1, SW8 Note2, SW9 Note3, U1 PLAYBACK, U2 74HC595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

Commit message: Add files via upload
Parts:
- added LS2: CDS-13138-SMT-TR, CDS-13138-SMT-TR:SPKR_CDS-13138-SMT-TR, symbol CDS-13138-SMT-TR:CDS-13138-SMT-TR
- added R8: 10k Ohms, Resistor_THT:R_Axial_DIN0204_L3.6mm_D1.6mm_P5.08mm_Horizontal, symbol Device:R
- added SW1, SW5, SW6: MODE, Button_Switch_THT:SW_Slide-03_Wuerth-WS-SLTV_10x2.5x6.4_P2.54mm, symbol Switch:SW_Wuerth_450301014042
- added SW10: SPEAKER, Button_Switch_THT:SW_Slide-03_Wuerth-WS-SLTV_10x2.5x6.4_P2.54mm, symbol Switch:SW_Wuerth_450301014042
- added SW4: CLEAR, Button_Switch_THT:SW_PUSH_6mm, symbol Switch:SW_Push
- C4: value 100uF -> 47uF
- R11, R12, R13: value 1000 -> 10k Ohms
- R2: value 5.1k Ohms -> 15k Ohms
Connections:
- net +5V: now also SW7.2, SW8.2, SW9.2, R8.1; no longer U2.12 (RCLK), U3.12 (RCLK), U4.12 (RCLK)
- net GND: now also SW3.1, LS2.M, SW4.1
- net tone1: now also SW6.3 (A); no longer SW7.2, U3.14 (SER)
- net tone2: now also SW5.3 (A); no longer SW8.2, U4.14 (SER)
- net tone3: now also SW1.3 (A); no longer SW9.2, U2.14 (SER)
- net at R22.2: now also SW10.1 (B); no longer LS1.1
- net at C1.2, U9.5 (CV): no longer SW3.1
- net at R11.1, SW7.1: now also SW6.2 (C)
- net at R13.1, SW9.1: now also SW1.2 (C)
- net CLR: now reaches U2.10 (~{SRCLR})
- net CLR: now also U3.10 (~{SRCLR}), U4.10 (~{SRCLR}), R8.2, SW4.2
- net at R12.1, SW8.1: now also SW5.2 (C)
- new net: LS1.1, SW10.2 (C)
- new net: LS2.P, SW10.3 (A)
- new net: SW6.1 (B), U3.14 (SER)
- new net: SW1.1 (B), U2.14 (SER)
- new net: SW5.1 (B), U4.14 (SER)
- no-connect marks 0 -> 28
Other:
- note added: "Clear Shift Registers"
- note added: "SISO Shift Register: Note 1 (A3)"
- note added: "SISO Shift Register: Note 2 (C4)"
- note added: "SISO Shift Register: Note 3 (D#4)"
- note removed: "SISO Shift Register: Note 1"
- note removed: "SISO Shift Register: Note 2"
- note removed: "SISO Shift Register: Note 3"
- moved on the sheet: BT1, C1, LS1, R11, R12, R13, R22, SW2, SW7, SW8, SW9
